File: pcb/soldriver.kicad_sch (KiCad schematic)
At the start: 66 parts, among them J1 1726480102, J10 705510001, J11 705510001, J12 705510001, J13 705510001, J14 705510001, J15 705510001, J16 n/a, J17 n/a, J18 2601-1102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

Commit message: switch to 2.2uF tantalum cap
Parts:
- C1: value 10u -> 2.2u; DIGIKEY_SKU 1276-CL31Y106KBKVPJECT-ND -> (none); MFR Samsung Electro-Mechanics -> KEMET; MOUSER_SKU (none) -> 80-T491A225K35ATAUTO; MPN CL31Y106KBKVPJE -> T491A225K035ATAUTO
Changed lines of the file:
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@@
 			)
 		)
-		(property "Description" "PTC self-resetting fuse, 200mA 30V"
+		(property "Description" "1206 PTC self-resetting fuse, 200mA 30V"
 			(at 158.75 128.27 0)
 			(effects
@@
 			)
 		)
-		(property "Description" "PTC self-resetting fuse, 200mA 30V"
+		(property "Description" "1206 PTC self-resetting fuse, 200mA 30V"
 			(at 158.75 140.97 0)
 			(effects
@@
 			)
 		)
-		(property "Description" "Ceramic cap 0.1uF 50V"
+		(property "Description" "0805 ceramic cap 0.1uF 50V"
 			(at 78.74 113.03 0)
 			(effects
@@
 			)
 		)
-		(property "Description" "PTC self-resetting fuse, 200mA 30V"
+		(property "Description" "1206 PTC self-resetting fuse, 200mA 30V"
 			(at 158.75 153.67 0)
 			(effects
@@
 			)
 		)
-		(property "Description" "SMD fuse 2A 30V"
+		(property "Description" "1206 SMD fuse fast acting 2A 63VDC"
 			(at 220.98 34.29 0)
 			(effects
@@
 			)
 		)
-		(property "Description" "PTC self-resetting fuse, 200mA 30V"
+		(property "Description" "1206 PTC self-resetting fuse, 200mA 30V"
 			(at 115.57 102.87 0)
 			(effects
@@
 			)
 		)
-		(property "Description" "Ceramic cap 0.1uF 50V"
+		(property "Description" "0805 ceramic cap 0.1uF 50V"
 			(at 78.74 158.75 0)
 			(effects
@@
 			)
 		)
-		(property "Description" "PTC self-resetting fuse, 200mA 30V"
+		(property "Description" "1206 PTC self-resetting fuse, 200mA 30V"
 			(at 115.57 140.97 0)
 			(effects
@@
 			)
 		)
-		(property "Description" "PTC self-resetting fuse, 200mA 30V"
+		(property "Description" "1206 PTC self-resetting fuse, 200mA 30V"
 			(at 158.75 90.17 0)
 			(effects
@@
 			)
 		)
-		(property "Description" "PTC self-resetting fuse, 200mA 30V"
+		(property "Description" "1206 PTC self-resetting fuse, 200mA 30V"
 			(at 115.57 153.67 0)
 			(effects
@@
 			)
 		)
-		(property "Description" "PTC self-resetting fuse, 200mA 30V"
+		(property "Description" "1206 PTC self-resetting fuse, 200mA 30V"
 			(at 158.75 102.87 0)
 			(effects
@@
 			)
 		)
-		(property "Value" "10u"
+		(property "Value" "2.2u"
 			(at 198.12 42.2909 0)
 			(effects
@@
 			)
 		)
-		(property "Description" "Ceramic cap 10uF 50V"
+		(property "Description" "1206 tantalum cap 35V 2.2uF"
 			(at 201.93 41.91 0)
 			(effects
@@
 			)
 		)
-		(property "DIGIKEY_SKU" "1276-CL31Y106KBKVPJECT-ND"
+		(property "DIGIKEY_SKU" ""
 			(at 201.93 41.91 0)
 			(effects
@@
 			)
 		)
-		(property "MFR" "Samsung Electro-Mechanics"
+		(property "MFR" "KEMET"
 			(at 201.93 41.91 0)
 			(effects
@@
 			)
 		)
-		(property "MOUSER_SKU" ""
+		(property "MOUSER_SKU" "80-T491A225K35ATAUTO"
 			(at 201.93 41.91 0)
 			(effects
@@
 			)
 		)
-		(property "MPN" "CL31Y106KBKVPJE"
+		(property "MPN" "T491A225K035ATAUTO"
 			(at 201.93 41.91 0)
 			(effects
@@
 			)
 		)
-		(property "Description" "PTC self-resetting fuse, 200mA 30V"
+		(property "Description" "1206 PTC self-resetting fuse, 200mA 30V"
 			(at 115.57 90.17 0)
 			(effects
@@
 			)
 		)
-		(property "Description" "PTC self-resetting fuse, 200mA 30V"
+		(property "Description" "1206 PTC self-resetting fuse, 200mA 30V"
 			(at 158.75 115.57 0)
 			(effects
@@
 			)
 		)
-		(property "Description" "PTC self-resetting fuse, 200mA 30V"
+		(property "Description" "1206 PTC self-resetting fuse, 200mA 30V"
 			(at 115.57 115.57 0)
 			(effects
@@
 			)
 		)
-		(property "Description" "PTC self-resetting fuse, 200mA 30V"
+		(property "Description" "1206 PTC self-resetting fuse, 200mA 30V"
 			(at 115.57 128.27 0)
 			(effects

Commit message: update DN12 schematic title block and add PDF
Other:
- title: CBEIO1 12-channel USB solenoid/relay driver -> UXIB-DN12 12-channel USB solenoid/relay driver
Changed lines of the file:
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@@
 	(paper "A4")
 	(title_block
-		(title "CBEIO1 12-channel USB solenoid/relay driver")
-		(date "2024-04-18")
-		(rev "4")
+		(title "UXIB-DN12 12-channel USB solenoid/relay driver")
+		(date "2024-10-08")
+		(rev "5")
 		(company "Bioengineering Platform, Chan Zuckerberg Biohub San Francisco")
 		(comment 1 "Greg Courville <greg.courville@czbiohub.org>")
